Commit message: fix: sensors attached to trunk via xacro include, real meshes, angle fix
- Use robot_with_sensors.xacro wrapper (proper xacro:include chain)
  instead of string injection — fixes sensors floating detached
- Real DAE meshes: lidar_3d_v1.dae + realsense.dae (from playground)
- Lidar pitch: 0.349 (positive = forward tilt in URDF convention)
- Positions: lidar at (0.15, 0, 0.10), camera at (0.27, 0, 0.08)

File: gazebo/models/go2/sensors.xacro (robot description, xacro)
@@ -1,29 +1,28 @@
 <?xml version="1.0"?>
 <!--
-  Vector OS Nano — Go2 external sensor xacro
-  Adds Livox MID-360 lidar + RealSense D435 to the Go2 URDF.
-  Include this after the base robot.xacro.
-  Sensor mounting matches real Go2 hardware (see reference photo):
-    - MID-360: back-mounted on custom bracket, ~20 deg forward tilt
-    - D435: front-facing at nose height, ~5 deg downward tilt
+  Vector OS Nano — Go2 external sensors
+  Adds Livox MID-360 lidar + RealSense D435 to Go2 URDF.
+  Sensor mounting matches real Go2 hardware:
+    - MID-360: shoulder-mounted behind head, 20 deg forward tilt
+    - D435: in front of MID-360, slight downward tilt
+  Uses real mesh files for visual representation.
 -->
 <robot xmlns:xacro="http://www.ros.org/wiki/xacro">
+  <!-- Mesh path — absolute to avoid fragile relative paths -->
+  <xacro:property name="sensor_mesh_dir"
+    value="/home/yusen/Desktop/vector_os_nano/gazebo/models/go2/meshes/sensors"/>
   <!-- ============================================================ -->
   <!-- Livox MID-360 LiDAR                                          -->
-  <!-- Mounted just behind the head, on top of shoulders.           -->
-  <!-- x=0.15 (behind head at x=0.29, above shoulder line)          -->
-  <!-- z=0.15 (shoulder top + bracket)                              -->
-  <!-- Tilted 20 deg forward for ground coverage.                   -->
+  <!-- Shoulder-mounted, just behind head, 20 deg forward tilt      -->
   <!-- ============================================================ -->
   <joint name="mid360_joint" type="fixed">
     <parent link="trunk"/>
     <child link="mid360_link"/>
-    <!-- Behind head, on shoulders, tilted 20 deg forward -->
-    <origin xyz="0.15 0.0 0.15" rpy="0 -0.349 0"/>
+    <origin xyz="0.15 0.0 0.10" rpy="0 0.349 0"/>
   </joint>
   <link name="mid360_link">
     <inertial>
-      <mass value="0.265"/>  <!-- MID-360 actual mass: 265g -->
-      <origin xyz="0 0 0" rpy="0 0 0"/>
+      <mass value="0.265"/>
+      <origin xyz="0 0 0.03" rpy="0 0 0"/>
       <inertia ixx="0.0002" ixy="0" ixz="0" iyy="0.0002" iyz="0" izz="0.0003"/>
     </inertial>
@@ -31,12 +30,9 @@
       <origin xyz="0 0 0" rpy="0 0 0"/>
       <geometry>
-        <cylinder radius="0.05" length="0.06"/>  <!-- MID-360 puck shape -->
+        <mesh filename="file://${sensor_mesh_dir}/lidar_3d_v1.dae" scale="1 1 1"/>
       </geometry>
-      <material name="mid360_gray">
-        <color rgba="0.3 0.3 0.3 1"/>
-      </material>
     </visual>
     <collision>
-      <origin xyz="0 0 0" rpy="0 0 0"/>
+      <origin xyz="0 0 0.03" rpy="0 0 0"/>
       <geometry>
         <cylinder radius="0.05" length="0.06"/>
@@ -62,5 +58,4 @@
             <samples>30</samples>
             <resolution>1</resolution>
-            <!-- MID-360 VFoV: -7 to +52 deg -->
             <min_angle>-0.122</min_angle>
             <max_angle>0.908</max_angle>
@@ -77,28 +72,22 @@
   <!-- ============================================================ -->
   <!-- RealSense D435 RGB-D Camera                                   -->
-  <!-- Mounted in front of MID-360, on the head/shoulder area.      -->
-  <!-- Slightly forward and lower than the lidar.                   -->
-  <!-- ~5 deg downward tilt for ground object visibility.           -->
+  <!-- In front of MID-360, on head, 5 deg downward tilt            -->
   <!-- ============================================================ -->
   <joint name="d435_joint" type="fixed">
     <parent link="trunk"/>
     <child link="d435_link"/>
-    <!-- In front of MID-360, on head area, 5 deg down -->
-    <origin xyz="0.27 0.0 0.12" rpy="0 0.087 0"/>
+    <origin xyz="0.27 0.0 0.08" rpy="0 0.087 0"/>
   </joint>
   <link name="d435_link">
     <inertial>
-      <mass value="0.072"/>  <!-- D435 actual mass: 72g -->
+      <mass value="0.072"/>
       <origin xyz="0 0 0" rpy="0 0 0"/>
       <inertia ixx="0.00005" ixy="0" ixz="0" iyy="0.00005" iyz="0" izz="0.00003"/>
     </inertial>
     <visual>
-      <origin xyz="0 0 0" rpy="0 0 0"/>
+      <origin xyz="0 0 0" rpy="0 0 1.5708"/>
       <geometry>
-        <box size="0.025 0.09 0.025"/>  <!-- D435 form factor -->
+        <mesh filename="file://${sensor_mesh_dir}/realsense.dae" scale="1 1 1"/>
       </geometry>
-      <material name="d435_silver">
-        <color rgba="0.7 0.7 0.7 1"/>
-      </material>
     </visual>
     <collision>
@@ -109,12 +98,4 @@
     </collision>
   </link>
-  <!-- D435 optical frame (Z forward, X right, Y down — camera convention) -->
-  <joint name="d435_optical_joint" type="fixed">
-    <parent link="d435_link"/>
-    <child link="d435_optical_frame"/>
-    <origin xyz="0 0 0" rpy="-1.5708 0 -1.5708"/>
-  </joint>
-  <link name="d435_optical_frame"/>
-  <!-- D435 RGB camera sensor -->
   <gazebo reference="d435_link">
     <sensor name="d435_rgb" type="camera">
@@ -125,5 +106,5 @@
       <visualize>false</visualize>
       <camera>
-        <horizontal_fov>1.20</horizontal_fov>  <!-- ~69 deg -->
+        <horizontal_fov>1.20</horizontal_fov>
         <image>
           <width>640</width>
@@ -135,15 +116,9 @@
           <far>15.0</far>
         </clip>
-        <noise>
-          <type>gaussian</type>
-          <mean>0.0</mean>
-          <stddev>0.005</stddev>
-        </noise>
-        <optical_frame_id>d435_optical_frame</optical_frame_id>
+        <optical_frame_id>d435_link</optical_frame_id>
         <camera_info_topic>/camera/camera_info</camera_info_topic>
       </camera>
     </sensor>
   </gazebo>
-  <!-- D435 depth camera sensor — separate sensor on same link -->
   <gazebo reference="d435_link">
     <sensor name="d435_depth" type="depth_camera">
@@ -164,9 +139,4 @@
           <far>10.0</far>
         </clip>
-        <noise>
-          <type>gaussian</type>
-          <mean>0.0</mean>
-          <stddev>0.002</stddev>
-        </noise>
       </camera>
     </sensor>
