Commit message: feat: E2E pipeline test + v1.8.0 release prep
- tests/e2e/test_explore_navigate_e2e.py: 16 tests covering
  MuJoCo load → explore → SceneGraph → navigate → room resolution
- FAR config validation tests (intensity threshold, decay, votes)
- progress.md updated to v1.8.0
- .gitignore: add *.ply
- Gazebo files committed as-is (archived backend)

File: gazebo/models/go2/robot_with_sensors.xacro (robot description, xacro)
@@ -1,20 +1,17 @@
 <?xml version="1.0"?>
 <!--
-  Vector OS Nano — Go2 with MID-360 + D435 sensors for Gazebo Harmonic.
-  Proper xacro:include chain so all links/joints are in the same robot model.
+  Go2 with standard gz_ros2_control + MID-360 + D435 sensors.
+  Uses effort-only command interface (standard gz_ros2_control plugin).
 -->
 <robot name="go2" xmlns:xacro="http://www.ros.org/wiki/xacro">
-  <xacro:arg name="DEBUG" default="false"/>
-  <xacro:arg name="GAZEBO" default="true"/>
-  <xacro:arg name="CLASSIC" default="false"/>
-  <!-- Base Go2 robot (includes legs, trunk, ros2_control, gazebo plugins) -->
+  <!-- Go2 constants + materials + leg macro from upstream -->
   <xacro:include filename="$(find go2_description)/xacro/const.xacro"/>
   <xacro:include filename="$(find go2_description)/xacro/materials.xacro"/>
   <xacro:include filename="$(find go2_description)/xacro/leg.xacro"/>
-  <xacro:include filename="$(find go2_description)/xacro/gazebo.xacro"/>
-  <!-- Robot structure (copied from robot.xacro to avoid double-include issues) -->
+  <!-- Our ros2_control config (standard gz_ros2_control, NOT custom gz_quadruped_hardware) -->
+  <xacro:include filename="gazebo_ros2_control.xacro"/>
+  <!-- Robot structure -->
   <link name="base">
     <visual>
-      <origin rpy="0 0 0" xyz="0 0 0"/>
       <geometry><box size="0.001 0.001 0.001"/></geometry>
     </visual>
@@ -27,5 +24,4 @@
   <link name="trunk">
     <visual>
-      <origin rpy="0 0 0" xyz="0 0 0"/>
       <geometry>
         <mesh filename="file://$(find go2_description)/meshes/trunk.dae" scale="1 1 1"/>
@@ -33,18 +29,5 @@
     </visual>
     <collision>
-      <origin rpy="0 0 0" xyz="0 0 0"/>
       <geometry><box size="${trunk_length} ${trunk_width} ${trunk_height}"/></geometry>
-    </collision>
-    <collision>
-      <origin rpy="0 0 0" xyz="0 0 0"/>
-      <geometry><box size="0.1881 0.04675 0.057"/></geometry>
-    </collision>
-    <collision>
-      <origin rpy="0 0 0" xyz="0.285 0 0.01"/>
-      <geometry><cylinder length="0.05" radius="0.045"/></geometry>
-    </collision>
-    <collision>
-      <origin rpy="0 0 0" xyz="0.293 0 -0.06"/>
-      <geometry><box size="0.047 0.047 0.047"/></geometry>
     </collision>
     <inertial>
@@ -63,15 +46,8 @@
     <inertial>
       <mass value="0.001"/>
-      <origin rpy="0 0 0" xyz="0 0 0"/>
       <inertia ixx="0.0001" ixy="0" ixz="0" iyy="0.0001" iyz="0" izz="0.0001"/>
     </inertial>
-    <visual>
-      <origin rpy="0 0 0" xyz="0 0 0"/>
-      <geometry><box size="0.001 0.001 0.001"/></geometry>
-    </visual>
-    <collision>
-      <origin rpy="0 0 0" xyz="0 0 0"/>
-      <geometry><box size=".001 .001 .001"/></geometry>
-    </collision>
+    <visual><geometry><box size="0.001 0.001 0.001"/></geometry></visual>
+    <collision><geometry><box size="0.001 0.001 0.001"/></geometry></collision>
   </link>
   <!-- Legs -->
@@ -80,5 +56,5 @@
   <xacro:leg name="RR" mirror="-1" mirror_dae="False" front_hind="-1" front_hind_dae="False"/>
   <xacro:leg name="RL" mirror="1" mirror_dae="True" front_hind="-1" front_hind_dae="False"/>
-  <!-- Vector OS Nano sensors (MID-360 + D435) — properly included in same robot -->
+  <!-- External sensors -->
   <xacro:include filename="sensors.xacro"/>
 </robot>
